File: DispenM/Balanza/Balanza.sch (KiCad schematic (older format))
At the start: 16 parts, among them J1 GPA/B0, J2 I2C, J3 INTA/INTB, J4 POWER, J5 BALANZA, SW1 SW_DIP_x03, SW2 SW_SPDT, U1 MCP23017_SP, U2 ESP32-DEVKITC-32D

Commit message: Nuevo programa
Parts:
- removed D1: NeoPixel_THT, Connector_PinHeader_2.54mm:PinHeader_1x04_P2.54mm_Vertical, symbol LED:NeoPixel_THT
- removed DS1: WC1602A, Display:WC1602A, symbol Display_Character:WC1602A
- removed J1: GPA/B0, Connector_PinHeader_2.54mm:PinHeader_1x09_P2.54mm_Vertical, symbol Connector_Generic:Conn_01x09
- removed J2: I2C, Connector_PinHeader_2.54mm:PinHeader_1x02_P2.54mm_Vertical, symbol Connector_Generic:Conn_01x02
- removed J3: INTA/INTB, Connector_PinHeader_2.54mm:PinHeader_1x02_P2.54mm_Vertical, symbol Connector_Generic:Conn_01x02
- removed J4: POWER, Connector_PinHeader_2.54mm:PinHeader_1x02_P2.54mm_Vertical, symbol Connector_Generic:Conn_01x02
- removed J5: BALANZA, MODULOS:ModuloHX711, symbol Connector_Generic:Conn_01x04
- removed R1: R, Resistor_THT:R_Axial_DIN0207_L6.3mm_D2.5mm_P10.16mm_Horizontal, symbol Device:R
- removed R2, R3, R4: 10k, Resistor_THT:R_Axial_DIN0207_L6.3mm_D2.5mm_P10.16mm_Horizontal, symbol Device:R
- removed RV1: R_POT, Potentiometer_THT:Potentiometer_ACP_CA9-V10_Vertical, symbol Device:R_POT
- removed SW1: SW_DIP_x03, Button_Switch_THT:SW_DIP_SPSTx03_Slide_9.78x9.8mm_W7.62mm_P2.54mm, symbol Switch:SW_DIP_x03
- removed SW2: SW_SPDT, Custom_Footprints:Slide_Switch_SPDT_ThroughHole, symbol Switch:SW_SPDT
- removed U1: MCP23017_SP, Package_DIP:DIP-28_W7.62mm, symbol Interface_Expansion:MCP23017_SP
- removed U2: ESP32-DEVKITC-32D, MODULOS:Esp32wroverD, symbol ESP32-DEVKITC-32D:ESP32-DEVKITC-32D
- added BOTO1, BOTO2, NiHALL1: Conn_01x03, Connector_PinHeader_2.54mm:PinHeader_1x03_P2.54mm_Vertical, symbol Connector_Generic:Conn_01x03
- added M1: Motor_Servo, Connector_PinHeader_2.54mm:PinHeader_1x03_P2.54mm_Vertical, symbol Motor:Motor_Servo
- added OLED2828: Conn_01x08, MODULOS:OLED128X128, symbol Connector_Generic:Conn_01x08
- added U1: LoRa32U4, MODULOS:Lora32U4, symbol LoRa32U4:LoRa32U4
- added U2: DS3231MZ, Package_SO:SOIC-8_3.9x4.9mm_P1.27mm, symbol Timer_RTC:DS3231MZ
Connections:
- net labels added: CS, DC, RST, SERVO, SI
- net labels removed: +5, D0, D4, D5, D6, D7, E, GPA0, GPA1, GPA2, GPA3, GPA4, GPA5, GPA6, GPA7, INTA, INTB, IO18, IO19, RS, RW
- wire segments 32 -> 7
- no-connect marks 5 -> 3
Other:
- note removed: "CONECTORES"
- note removed: "LCD I2C"
