File: DispenM/Balanza/Dispen2/Dispen2.kicad_pcb (KiCad board)
At the start: 2 copper layers, 66.2 x 91.2 mm, 7 parts, among them M1 Motor_Servo, U1 LoRa32U4, U2 DS3231MZ

Commit message: Correccion de plano
Parts:
- added BT1: 9V, TerminalBlock_Phoenix:TerminalBlock_Phoenix_MKDS-1,5-2-5.08_1x02_P5.08mm_Horizontal, F.Cu at (200.0, -4.40)
- added D1: 1N4001, Diode_THT:D_DO-41_SOD81_P3.81mm_Vertical_KathodeUp, F.Cu at (137.2, 19.6)
- added R1: 100, Resistor_THT:R_Axial_DIN0207_L6.3mm_D2.5mm_P10.16mm_Horizontal, F.Cu at (199.8, 5.20)
- added R2: 180, Resistor_THT:R_Axial_DIN0207_L6.3mm_D2.5mm_P10.16mm_Horizontal, F.Cu at (195.2, 15.4)
- added R3: 100, Resistor_THT:R_Axial_DIN0207_L6.3mm_D2.5mm_P10.16mm_Horizontal, F.Cu at (199.2, 21.0)
- added R4: 220, Resistor_THT:R_Axial_DIN0207_L6.3mm_D2.5mm_P10.16mm_Horizontal, F.Cu at (195.2, 31.0)
- moved BOTO1 0.05 mm to (180.2, 4.00)
Connections:
- U1 pad 10: SERVO -> (no net)
- U1 pad 5: RST -> (no net)
- U1 pad GND: GND -> (no net)
Routing:
- net +3V3: track 95.7 -> 195.1 mm
- net Net-(BT1-Pad2): track 0.00 -> 45.0 mm
- net +5V: track 159.7 -> 197.0 mm
- net Net-(BT1-Pad1): track 0.00 -> 9.68 mm
- net GND: track 171.5 -> 173.9 mm
- net Net-(BOTO1-Pad1): track 37.3 -> 38.2 mm
Other:
- board size 66.2 x 91.2 mm -> 71.8 x 91.2 mm

Commit message: Actualizacion software y pcb
Parts:
- moved U1 0.40 mm to (144.4, -9.80)
Connections:
- U1 pad 6: Net-(BOTO2-Pad1) -> (no net)
- U1 pad 9: Net-(BOTO1-Pad1) -> (no net)
Routing:
- net +5V: track 197.0 -> 211.8 mm

Commit message: Correccion pcb
Parts:
- removed BT1: 9V, TerminalBlock_Phoenix:TerminalBlock_Phoenix_MKDS-1,5-2-5.08_1x02_P5.08mm_Horizontal
- removed R1, R3: 100, Resistor_THT:R_Axial_DIN0207_L6.3mm_D2.5mm_P10.16mm_Horizontal
- removed R2: 180, Resistor_THT:R_Axial_DIN0207_L6.3mm_D2.5mm_P10.16mm_Horizontal
- removed R4: 220, Resistor_THT:R_Axial_DIN0207_L6.3mm_D2.5mm_P10.16mm_Horizontal
- moved BOTO1 3.60 mm to (183.8, 4.00)
- moved D1 3.60 mm to (140.8, 19.6)
- moved BOTO2 3.60 mm to (178.3, 4.00)
- moved M1 3.60 mm to (178.6, 15.8)
- moved NiHALL1 3.60 mm to (142.6, 7.50)
- moved OLED1 3.60 mm to (153.6, 67.8)
- moved U1 3.60 mm to (148.0, -9.80)
- moved U2 3.60 mm to (199.6, 40.5)
Connections:
- U1 pad 5V: +5V -> (no net)
- U1 pad GND: (no net) -> GND
Routing:
- net +3V3: track 195.1 -> 104.4 mm
- net +5V: track 211.8 -> 126.9 mm
- net Net-(BT1-Pad2): track 45.0 -> 0.00 mm
- net GND: track 173.9 -> 158.7 mm
- net Net-(BT1-Pad1): track 9.68 -> 0.00 mm
Other:
- board size 71.8 x 91.2 mm -> 69.8 x 91.2 mm

Commit message: Cambio de fuente
Parts:
- added J1: Conn_01x02, TerminalBlock_Phoenix:TerminalBlock_Phoenix_MKDS-1,5-2_1x02_P5.00mm_Horizontal, F.Cu at (202.8, -4.94)
- added U3: LD1117S33TR_SOT223, Package_TO_SOT_THT:TO-220-3_Vertical, F.Cu at (198.0, 18.4)
- added U4: LM7805_TO220, Package_TO_SOT_THT:TO-220-3_Vertical, F.Cu at (203.0, 5.87)
Connections:
- U1 pad GND: GND -> (no net)
Routing:
- net +3V3: track 104.4 -> 173.8 mm
- net +5V: track 126.9 -> 172.1 mm
- net Net-(J1-Pad1): track 0.00 -> 12.8 mm
Other:
- board size 69.8 x 91.2 mm -> 83.8 x 91.2 mm

Commit message: Ok sensor Hu
Parts:
- moved D1 37.3 mm to (147.0, 56.4)
- moved U2 11.0 mm to (210.6, 40.0)
- moved U3 4.71 mm to (202.7, 18.7), turned to 180 degrees
- moved NiHALL1 1.53 mm to (142.8, 9.01)
- moved U4 0.21 mm to (202.8, 5.84)
Connections:
- NiHALL1 pad 2: GND -> +5V
- NiHALL1 pad 3: +5V -> GND
- U3 pad 2: +5V -> +3V3
- U3 pad 3: +3V3 -> +5V
- U4 pad 1: +5V -> Net-(J1-Pad1)
- U4 pad 3: Net-(J1-Pad1) -> +5V
Routing:
- net GND: track 158.4 -> 0.00 mm
- net +5V: track 172.1 -> 235.3 mm
- net +3V3: track 173.8 -> 187.8 mm
- net SDA: track 24.4 -> 31.7 mm
- net SCL: track 38.6 -> 36.5 mm
- net Net-(J1-Pad1): track 12.8 -> 10.8 mm
- net Net-(NiHALL1-Pad1): track 8.48 -> 7.68 mm

Commit message: nuevo circuito
nuevo circuito
Parts:
- added CABLE1: R, Resistor_THT:R_Axial_DIN0411_L9.9mm_D3.6mm_P20.32mm_Horizontal, F.Cu at (203.8, 14.1)
- added CABLE2: R, Resistor_THT:R_Axial_DIN0411_L9.9mm_D3.6mm_P25.40mm_Horizontal, F.Cu at (191.9, 51.1)
Routing:
- net GND: track 0.00 -> 45.7 mm
Changed lines of the file:
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@@
     (thickness 1.6)
     (drawings 4)
-    (tracks 129)
+    (tracks 131)
     (zones 0)
-    (modules 11)
+    (modules 13)
     (nets 23)
   )
@@
     (mod_text_size 1 1)
     (mod_text_width 0.15)
-    (pad_size 1.5 2.5)
-    (pad_drill 1.1)
+    (pad_size 2.5 1.7)
+    (pad_drill 1)
     (pad_to_mask_clearance 0)
     (aux_axis_origin 0 0)
@@
     (add_net SERVO)
     (add_net SI)
+  )
+  (module Resistor_THT:R_Axial_DIN0411_L9.9mm_D3.6mm_P20.32mm_Horizontal (layer F.Cu)
+    (at 203.83 14.09 180)
+    (descr "Resistor, Axial_DIN0411 series, Axial, Horizontal, pin pitch=20.32mm, 1W, length*diameter=9.9*3.6mm^2")
+    (tags "Resistor Axial_DIN0411 series Axial Horizontal pin pitch 20.32mm 1W length 9.9mm diameter 3.6mm")
+    (fp_text reference CABLE1 (at 10.16 -2.92) (layer F.SilkS)
+      (effects (font (size 1 1) (thickness 0.15)))
+    )
+    (fp_text value R (at 10.16 2.92) (layer F.Fab)
+      (effects (font (size 1 1) (thickness 0.15)))
+    )
+    (fp_line (start 21.77 -2.05) (end -1.45 -2.05) (layer F.CrtYd) (width 0.05))
+    (fp_line (start 21.77 2.05) (end 21.77 -2.05) (layer F.CrtYd) (width 0.05))
+    (fp_line (start -1.45 2.05) (end 21.77 2.05) (layer F.CrtYd) (width 0.05))
+    (fp_line (start -1.45 -2.05) (end -1.45 2.05) (layer F.CrtYd) (width 0.05))
+    (fp_line (start 18.88 0) (end 15.23 0) (layer F.SilkS) (width 0.12))
+    (fp_line (start 1.44 0) (end 5.09 0) (layer F.SilkS) (width 0.12))
+    (fp_line (start 15.23 -1.92) (end 5.09 -1.92) (layer F.SilkS) (width 0.12))
+    (fp_line (start 15.23 1.92) (end 15.23 -1.92) (layer F.SilkS) (width 0.12))
+    (fp_line (start 5.09 1.92) (end 15.23 1.92) (layer F.SilkS) (width 0.12))
+    (fp_line (start 5.09 -1.92) (end 5.09 1.92) (layer F.SilkS) (width 0.12))
+    (fp_line (start 20.32 0) (end 15.11 0) (layer F.Fab) (width 0.1))
+    (fp_line (start 0 0) (end 5.21 0) (layer F.Fab) (width 0.1))
+    (fp_line (start 15.11 -1.8) (end 5.21 -1.8) (layer F.Fab) (width 0.1))
+    (fp_line (start 15.11 1.8) (end 15.11 -1.8) (layer F.Fab) (width 0.1))
+    (fp_line (start 5.21 1.8) (end 15.11 1.8) (layer F.Fab) (width 0.1))
+    (fp_line (start 5.21 -1.8) (end 5.21 1.8) (layer F.Fab) (width 0.1))
+    (fp_text user %R (at 9.75 0.28) (layer F.Fab)
+      (effects (font (size 1 1) (thickness 0.15)))
+    )
+    (pad 2 thru_hole oval (at 20.32 0 180) (size 2.4 2.4) (drill 1.2) (layers *.Cu *.Mask)
+      (net 1 GND))
+    (pad 1 thru_hole circle (at 0 0 180) (size 2.4 2.4) (drill 1.2) (layers *.Cu *.Mask)
+      (net 1 GND))
+    (model ${KISYS3DMOD}/Resistor_THT.3dshapes/R_Axial_DIN0411_L9.9mm_D3.6mm_P20.32mm_Horizontal.wrl
+      (at (xyz 0 0 0))
+      (scale (xyz 1 1 1))
+      (rotate (xyz 0 0 0))
+    )
+  )
+  (module Resistor_THT:R_Axial_DIN0411_L9.9mm_D3.6mm_P25.40mm_Horizontal (layer F.Cu)
+    (at 191.87 51.11 90)
+    (descr "Resistor, Axial_DIN0411 series, Axial, Horizontal, pin pitch=25.4mm, 1W, length*diameter=9.9*3.6mm^2")
+    (tags "Resistor Axial_DIN0411 series Axial Horizontal pin pitch 25.4mm 1W length 9.9mm diameter 3.6mm")
+    (fp_text reference CABLE2 (at 10.16 -2.92 90) (layer F.SilkS)
+      (effects (font (size 1 1) (thickness 0.15)))
+    )
+    (fp_text value R (at 10.16 2.92 90) (layer F.Fab)
+      (effects (font (size 1 1) (thickness 0.15)))
+    )
+    (fp_line (start 26.85 -2.05) (end -1.45 -2.05) (layer F.CrtYd) (width 0.05))
+    (fp_line (start 26.85 2.05) (end 26.85 -2.05) (layer F.CrtYd) (width 0.05))
+    (fp_line (start -1.45 2.05) (end 26.85 2.05) (layer F.CrtYd) (width 0.05))
+    (fp_line (start -1.45 -2.05) (end -1.45 2.05) (layer F.CrtYd) (width 0.05))
+    (fp_line (start 23.96 0) (end 17.77 0) (layer F.SilkS) (width 0.12))
+    (fp_line (start 1.44 0) (end 7.63 0) (layer F.SilkS) (width 0.12))
+    (fp_line (start 17.77 -1.92) (end 7.63 -1.92) (layer F.SilkS) (width 0.12))
+    (fp_line (start 17.77 1.92) (end 17.77 -1.92) (layer F.SilkS) (width 0.12))
+    (fp_line (start 7.63 1.92) (end 17.77 1.92) (layer F.SilkS) (width 0.12))
+    (fp_line (start 7.63 -1.92) (end 7.63 1.92) (layer F.SilkS) (width 0.12))
+    (fp_line (start 25.4 0) (end 17.65 0) (layer F.Fab) (width 0.1))
+    (fp_line (start 0 0) (end 7.75 0) (layer F.Fab) (width 0.1))
+    (fp_line (start 17.65 -1.8) (end 7.75 -1.8) (layer F.Fab) (width 0.1))
+    (fp_line (start 17.65 1.8) (end 17.65 -1.8) (layer F.Fab) (width 0.1))
+    (fp_line (start 7.75 1.8) (end 17.65 1.8) (layer F.Fab) (width 0.1))
+    (fp_line (start 7.75 -1.8) (end 7.75 1.8) (layer F.Fab) (width 0.1))
+    (fp_text user %R (at 10.16 0 90) (layer F.Fab)
+      (effects (font (size 1 1) (thickness 0.15)))
+    )
+    (pad 2 thru_hole oval (at 25.4 0 90) (size 2.4 2.4) (drill 1.2) (layers *.Cu *.Mask)
+      (net 1 GND))
+    (pad 1 thru_hole circle (at 0 0 90) (size 2.4 2.4) (drill 1.2) (layers *.Cu *.Mask)
+      (net 1 GND))
+    (model ${KISYS3DMOD}/Resistor_THT.3dshapes/R_Axial_DIN0411_L9.9mm_D3.6mm_P25.40mm_Horizontal.wrl
+      (at (xyz 0 0 0))
+      (scale (xyz 1 1 1))
+      (rotate (xyz 0 0 0))
+    )
   )
   (module MODULOS:DS3231MH (layer F.Cu)
@@
   (gr_line (start 132 -10.75) (end 215.77 -10.75) (layer Edge.Cuts) (width 0.05))
   (segment (start 149.3 4.57) (end 149.67 4.57) (width 0.5) (layer F.Cu) (net 0))
+  (segment (start 191.87 25.71) (end 191.87 51.11) (width 0.5) (layer B.Cu) (net 1))
+  (segment (start 183.51 14.09) (end 203.83 14.09) (width 0.5) (layer B.Cu) (net 1))
   (segment (start 178.35 6.54) (end 183.85 6.54) (width 0.5) (layer F.Cu) (net 2))
   (segment (start 176.39 6.54) (end 178.35 6.54) (width 0.5) (layer F.Cu) (net 2))
