File: DispenM/Balanza/Dispen2/Dispen2.sch (KiCad schematic (older format))
At the start: 7 parts, among them M1 Motor_Servo, U1 LoRa32U4, U2 DS3231MZ

Commit message: Correccion de plano
Parts:
- added BT1: 9V, TerminalBlock_Phoenix:TerminalBlock_Phoenix_MKDS-1,5-2-5.08_1x02_P5.08mm_Horizontal, symbol Device:Battery
- added D1: 1N4001, Diode_THT:D_DO-41_SOD81_P3.81mm_Vertical_KathodeUp, symbol Diode:1N4001
- added R1, R3: 100, Resistor_THT:R_Axial_DIN0207_L6.3mm_D2.5mm_P10.16mm_Horizontal, symbol Device:R
- added R2: 180, Resistor_THT:R_Axial_DIN0207_L6.3mm_D2.5mm_P10.16mm_Horizontal, symbol Device:R
- added R4: 220, Resistor_THT:R_Axial_DIN0207_L6.3mm_D2.5mm_P10.16mm_Horizontal, symbol Device:R
Connections:
- net +3V3: now also U1.~ (RST), R3.2, R4.1
- net +5V: now also D1.1 (K), R1.2, R2.1, R3.1
- net GND: now also D1.2 (A)
- new net: BT1.1 (+), R1.1
- new net: BT1.2 (-), R2.2, R4.2
- no-connect marks 16 -> 18
Other:
- moved on the sheet: OLED1
Changed lines of the file:
@@
 L Connector_Generic:Conn_01x08 OLED1
 U 1 1 6484BF16
-P 3900 3950
-F 0 "OLED1" H 3818 4467 50  0000 C CNN
-F 1 "Conn_01x08" H 3818 4376 50  0000 C CNN
-F 2 "MODULOS:OLED128X128" H 3900 3950 50  0001 C CNN
-F 3 "~" H 3900 3950 50  0001 C CNN
-	1    3900 3950
+P 3150 3650
+F 0 "OLED1" H 3068 4167 50  0000 C CNN
+F 1 "Conn_01x08" H 3068 4076 50  0000 C CNN
+F 2 "MODULOS:OLED128X128" H 3150 3650 50  0001 C CNN
+F 3 "~" H 3150 3650 50  0001 C CNN
+	1    3150 3650
 	-1   0    0    -1
 $EndComp
@@
 L power:+3.3V #PWR0101
 U 1 1 64852F69
-P 4100 3650
-F 0 "#PWR0101" H 4100 3500 50  0001 C CNN
-F 1 "+3.3V" V 4115 3778 50  0000 L CNN
-F 2 "" H 4100 3650 50  0001 C CNN
-F 3 "" H 4100 3650 50  0001 C CNN
-	1    4100 3650
+P 3350 3350
+F 0 "#PWR0101" H 3350 3200 50  0001 C CNN
+F 1 "+3.3V" V 3365 3478 50  0000 L CNN
+F 2 "" H 3350 3350 50  0001 C CNN
+F 3 "" H 3350 3350 50  0001 C CNN
+	1    3350 3350
 	0    1    1    0
 $EndComp
@@
 L power:+5V #PWR0106
 U 1 1 6485769F
-P 4100 3750
-F 0 "#PWR0106" H 4100 3600 50  0001 C CNN
-F 1 "+5V" V 4115 3878 50  0000 L CNN
-F 2 "" H 4100 3750 50  0001 C CNN
-F 3 "" H 4100 3750 50  0001 C CNN
-	1    4100 3750
+P 3850 3350
+F 0 "#PWR0106" H 3850 3200 50  0001 C CNN
+F 1 "+5V" V 3865 3478 50  0000 L CNN
+F 2 "" H 3850 3350 50  0001 C CNN
+F 3 "" H 3850 3350 50  0001 C CNN
+	1    3850 3350
 	0    1    1    0
 $EndComp
@@
 L power:GND #PWR0108
 U 1 1 6485B27F
-P 4100 3850
-F 0 "#PWR0108" H 4100 3600 50  0001 C CNN
-F 1 "GND" V 4105 3722 50  0000 R CNN
-F 2 "" H 4100 3850 50  0001 C CNN
-F 3 "" H 4100 3850 50  0001 C CNN
-	1    4100 3850
+P 3850 3650
+F 0 "#PWR0108" H 3850 3400 50  0001 C CNN
+F 1 "GND" V 3855 3522 50  0000 R CNN
+F 2 "" H 3850 3650 50  0001 C CNN
+F 3 "" H 3850 3650 50  0001 C CNN
+	1    3850 3650
 	0    -1   -1   0
 $EndComp
@@
 Wire Wire Line
 	4600 2750 4050 2750
-Text GLabel 4100 3950 2    50   Input ~ 0
+Text GLabel 3350 3650 2    50   Input ~ 0
 RST
-Text GLabel 4100 4050 2    50   Input ~ 0
+Text GLabel 3350 3750 2    50   Input ~ 0
 SCK
-Text GLabel 4100 4150 2    50   Input ~ 0
+Text GLabel 3350 3850 2    50   Input ~ 0
 SI
-Text GLabel 4100 4250 2    50   Input ~ 0
+Text GLabel 3350 3950 2    50   Input ~ 0
 CS
-Text GLabel 4100 4350 2    50   Input ~ 0
+Text GLabel 3350 4050 2    50   Input ~ 0
 DC
 Wire Wire Line
 	6200 4000 6550 4000
-Wire Wire Line
-	5800 3450 6550 3450
 NoConn ~ 5800 3250
 NoConn ~ 5800 3150
@@
 NoConn ~ 5800 2850
 NoConn ~ 4600 2350
-NoConn ~ 4600 2450
 NoConn ~ 4600 2550
 NoConn ~ 4600 3550
@@
 NoConn ~ 4600 3850
 NoConn ~ 6400 1750
+$Comp
+L Device:Battery BT1
+U 1 1 64B82FDD
+P 3200 1450
+F 0 "BT1" H 3308 1496 50  0000 L CNN
+F 1 "9V" H 3250 1300 50  0000 L CNN
+F 2 "TerminalBlock_Phoenix:TerminalBlock_Phoenix_MKDS-1,5-2-5.08_1x02_P5.08mm_Horizontal" V 3200 1510 50  0001 C CNN
+F 3 "~" V 3200 1510 50  0001 C CNN
+	1    3200 1450
+	1    0    0    -1
+$EndComp
+$Comp
+L Device:R R1
+U 1 1 64B83CB1
+P 3550 1300
+F 0 "R1" H 3620 1346 50  0000 L CNN
+F 1 "100" H 3620 1255 50  0000 L CNN
+F 2 "Resistor_THT:R_Axial_DIN0207_L6.3mm_D2.5mm_P10.16mm_Horizontal" V 3480 1300 50  0001 C CNN
+F 3 "~" H 3550 1300 50  0001 C CNN
+	1    3550 1300
+	1    0    0    -1
+$EndComp
+$Comp
+L Diode:1N4001 D1
+U 1 1 64B84623
+P 3850 3500
+F 0 "D1" V 3804 3580 50  0000 L CNN
+F 1 "1N4001" V 3895 3580 50  0000 L CNN
+F 2 "Diode_THT:D_DO-41_SOD81_P3.81mm_Vertical_KathodeUp" H 3850 3325 50  0001 C CNN
+F 3 "http://www.vishay.com/docs/88503/1n4001.pdf" H 3850 3500 50  0001 C CNN
+	1    3850 3500
+	0    1    1    0
+$EndComp
+Wire Wire Line
+	3850 3350 3750 3350
+Wire Wire Line
+	3750 3350 3750 3450
+Wire Wire Line
+	3750 3450 3350 3450
+Connection ~ 3850 3350
+Wire Wire Line
+	3350 3550 3750 3550
+Wire Wire Line
+	3750 3550 3750 3650
+Wire Wire Line
+	3750 3650 3850 3650
+Connection ~ 3850 3650
+$Comp
+L Device:R R2
+U 1 1 64B8C058
+P 3550 1700
+F 0 "R2" H 3620 1746 50  0000 L CNN
+F 1 "180" H 3620 1655 50  0000 L CNN
+F 2 "Resistor_THT:R_Axial_DIN0207_L6.3mm_D2.5mm_P10.16mm_Horizontal" V 3480 1700 50  0001 C CNN
+F 3 "~" H 3550 1700 50  0001 C CNN
+	1    3550 1700
+	1    0    0    -1
+$EndComp
+$Comp
+L Device:R R4
+U 1 1 64B8C9C1
+P 3900 2000
+F 0 "R4" H 3970 2046 50  0000 L CNN
+F 1 "220" H 3970 1955 50  0000 L CNN
+F 2 "Resistor_THT:R_Axial_DIN0207_L6.3mm_D2.5mm_P10.16mm_Horizontal" V 3830 2000 50  0001 C CNN
+F 3 "~" H 3900 2000 50  0001 C CNN
+	1    3900 2000
+	1    0    0    -1
+$EndComp
+Wire Wire Line
+	3200 1250 3200 1150
+Wire Wire Line
+	3200 1650 3200 1850
+Wire Wire Line
+	3200 1150 3550 1150
+Wire Wire Line
+	3200 1850 3550 1850
+Wire Wire Line
+	3550 1850 3550 2150
+Wire Wire Line
+	3550 2150 3900 2150
+Connection ~ 3550 1850
+Wire Wire Line
+	3550 1500 3550 1450
+Wire Wire Line
+	3550 1550 3550 1500
+Connection ~ 3550 1500
+$Comp
+L Device:R R3
+U 1 1 64B8C357
+P 3900 1650
+F 0 "R3" H 3970 1696 50  0000 L CNN
+F 1 "100" H 3970 1605 50  0000 L CNN
+F 2 "Resistor_THT:R_Axial_DIN0207_L6.3mm_D2.5mm_P10.16mm_Horizontal" V 3830 1650 50  0001 C CNN
+F 3 "~" H 3900 1650 50  0001 C CNN
+	1    3900 1650
+	1    0    0    -1
+$EndComp
+Wire Wire Line
+	3550 1500 3900 1500
+Wire Wire Line
+	3900 1800 3900 1850
+$Comp
+L power:+5V #PWR0115
+U 1 1 64B93850
+P 3550 1500
+F 0 "#PWR0115" H 3550 1350 50  0001 C CNN
+F 1 "+5V" V 3550 1600 50  0000 L CNN
+F 2 "" H 3550 1500 50  0001 C CNN
+F 3 "" H 3550 1500 50  0001 C CNN
+	1    3550 1500
+	0    -1   -1   0
+$EndComp
+$Comp
+L power:+3.3V #PWR0116
+U 1 1 64B93E40
+P 3900 1800
+F 0 "#PWR0116" H 3900 1650 50  0001 C CNN
+F 1 "+3.3V" V 3915 1928 50  0000 L CNN
+F 2 "" H 3900 1800 50  0001 C CNN
+F 3 "" H 3900 1800 50  0001 C CNN
+	1    3900 1800
+	0    1    1    0
+$EndComp
+Connection ~ 3900 1800
+$Comp
+L power:+3.3V #PWR0117
+U 1 1 64B94797
+P 4600 2450
+F 0 "#PWR0117" H 4600 2300 50  0001 C CNN
+F 1 "+3.3V" V 4615 2578 50  0000 L CNN
+F 2 "" H 4600 2450 50  0001 C CNN
+F 3 "" H 4600 2450 50  0001 C CNN
+	1    4600 2450
+	0    -1   -1   0
+$EndComp
+Wire Wire Line
+	5800 3450 6550 3450
+NoConn ~ 4600 2850
+NoConn ~ 4600 2950
+NoConn ~ 4600 3050
 $EndSCHEMATC

Commit message: Actualizacion software y pcb
Connections:
- net +5V: now also U1.~ (RST)
Other:
- moved on the sheet: BOTO1, M1, U2
Changed lines of the file:
@@
 $EndDescr
-$Comp
-L LoRa32U4:LoRa32U4 U1
-U 1 1 64849BFA
-P 5200 2750
-F 0 "U1" H 5200 3515 50  0000 C CNN
-F 1 "LoRa32U4" H 5200 3424 50  0000 C CNN
-F 2 "MODULOS:Lora32U4" H 5200 2750 50  0001 C CNN
-F 3 "" H 5200 2750 50  0001 C CNN
-	1    5200 2750
-	1    0    0    -1
-$EndComp
 $Comp
 L Motor:Motor_Servo M1
 U 1 1 6484B47B
-P 6550 3000
-F 0 "M1" H 6450 3000 50  0000 L CNN
-F 1 "Motor_Servo" H 6400 2900 50  0000 L CNN
-F 2 "Connector_PinHeader_2.54mm:PinHeader_1x03_P2.54mm_Vertical" H 6550 2810 50  0001 C CNN
-F 3 "http://forums.parallax.com/uploads/attachments/46831/74481.png" H 6550 2810 50  0001 C CNN
-	1    6550 3000
+P 6650 2450
+F 0 "M1" H 6550 2450 50  0000 L CNN
+F 1 "Motor_Servo" H 6500 2350 50  0000 L CNN
+F 2 "Connector_PinHeader_2.54mm:PinHeader_1x03_P2.54mm_Vertical" H 6650 2260 50  0001 C CNN
+F 3 "http://forums.parallax.com/uploads/attachments/46831/74481.png" H 6650 2260 50  0001 C CNN
+	1    6650 2450
 	1    0    0    -1
 $EndComp
@@
 L Timer_RTC:DS3231MZ U2
 U 1 1 6484C580
-P 6500 2150
-F 0 "U2" H 6500 2200 50  0000 C CNN
-F 1 "DS3231MZ" H 6300 2100 50  0000 C CNN
-F 2 "MODULOS:DS3231MH" H 6500 1650 50  0001 C CNN
-F 3 "http://datasheets.maximintegrated.com/en/ds/DS3231M.pdf" H 6500 1550 50  0001 C CNN
-	1    6500 2150
+P 6600 1500
+F 0 "U2" H 6600 1550 50  0000 C CNN
+F 1 "DS3231MZ" H 6400 1450 50  0000 C CNN
+F 2 "MODULOS:DS3231MH" H 6600 1000 50  0001 C CNN
+F 3 "http://datasheets.maximintegrated.com/en/ds/DS3231M.pdf" H 6600 900 50  0001 C CNN
+	1    6600 1500
 	1    0    0    -1
 $EndComp
@@
 L Connector_Generic:Conn_01x03 BOTO1
 U 1 1 6484ED92
-P 6750 3550
-F 0 "BOTO1" H 6668 3867 50  0000 C CNN
-F 1 "Conn_01x03" H 6668 3776 50  0000 C CNN
-F 2 "Connector_PinHeader_2.54mm:PinHeader_1x03_P2.54mm_Vertical" H 6750 3550 50  0001 C CNN
-F 3 "~" H 6750 3550 50  0001 C CNN
-	1    6750 3550
+P 6750 3350
+F 0 "BOTO1" H 6668 3667 50  0000 C CNN
+F 1 "Conn_01x03" H 6668 3576 50  0000 C CNN
+F 2 "Connector_PinHeader_2.54mm:PinHeader_1x03_P2.54mm_Vertical" H 6750 3350 50  0001 C CNN
+F 3 "~" H 6750 3350 50  0001 C CNN
+	1    6750 3350
 	1    0    0    -1
 $EndComp
@@
 L power:+3.3V #PWR0102
 U 1 1 648545ED
-P 6550 3550
-F 0 "#PWR0102" H 6550 3400 50  0001 C CNN
-F 1 "+3.3V" V 6565 3678 50  0000 L CNN
-F 2 "" H 6550 3550 50  0001 C CNN
-F 3 "" H 6550 3550 50  0001 C CNN
-	1    6550 3550
+P 6550 3350
+F 0 "#PWR0102" H 6550 3200 50  0001 C CNN
+F 1 "+3.3V" V 6565 3478 50  0000 L CNN
+F 2 "" H 6550 3350 50  0001 C CNN
+F 3 "" H 6550 3350 50  0001 C CNN
+	1    6550 3350
 	0    -1   -1   0
 $EndComp
@@
 L power:+5V #PWR0104
 U 1 1 64856200
-P 6250 3000
-F 0 "#PWR0104" H 6250 2850 50  0001 C CNN
-F 1 "+5V" V 6265 3128 50  0000 L CNN
-F 2 "" H 6250 3000 50  0001 C CNN
-F 3 "" H 6250 3000 50  0001 C CNN
-	1    6250 3000
+P 6350 2450
+F 0 "#PWR0104" H 6350 2300 50  0001 C CNN
+F 1 "+5V" V 6365 2578 50  0000 L CNN
+F 2 "" H 6350 2450 50  0001 C CNN
+F 3 "" H 6350 2450 50  0001 C CNN
+	1    6350 2450
 	0    -1   -1   0
 $EndComp
@@
 L power:+5V #PWR0105
 U 1 1 64856E0D
-P 6500 1750
-F 0 "#PWR0105" H 6500 1600 50  0001 C CNN
-F 1 "+5V" H 6515 1923 50  0000 C CNN
-F 2 "" H 6500 1750 50  0001 C CNN
-F 3 "" H 6500 1750 50  0001 C CNN
-	1    6500 1750
+P 6600 1100
+F 0 "#PWR0105" H 6600 950 50  0001 C CNN
+F 1 "+5V" H 6615 1273 50  0000 C CNN
+F 2 "" H 6600 1100 50  0001 C CNN
+F 3 "" H 6600 1100 50  0001 C CNN
+	1    6600 1100
 	1    0    0    -1
 $EndComp
@@
 	0    1    1    0
 $EndComp
-NoConn ~ 7000 1950
-NoConn ~ 7000 2250
-NoConn ~ 6000 2350
+NoConn ~ 7100 1300
+NoConn ~ 7100 1600
+NoConn ~ 6100 1700
 $Comp
 L power:GND #PWR0107
@@
 L power:GND #PWR0109
 U 1 1 6485B66E
-P 6500 2550
-F 0 "#PWR0109" H 6500 2300 50  0001 C CNN
-F 1 "GND" H 6505 2377 50  0000 C CNN
-F 2 "" H 6500 2550 50  0001 C CNN
-F 3 "" H 6500 2550 50  0001 C CNN
-	1    6500 2550
+P 6600 1900
+F 0 "#PWR0109" H 6600 1650 50  0001 C CNN
+F 1 "GND" H 6605 1727 50  0000 C CNN
+F 2 "" H 6600 1900 50  0001 C CNN
+F 3 "" H 6600 1900 50  0001 C CNN
+	1    6600 1900
 	1    0    0    -1
 $EndComp
@@
 L power:GND #PWR0110
 U 1 1 6485BFB9
-P 6550 3650
-F 0 "#PWR0110" H 6550 3400 50  0001 C CNN
-F 1 "GND" V 6555 3522 50  0000 R CNN
-F 2 "" H 6550 3650 50  0001 C CNN
-F 3 "" H 6550 3650 50  0001 C CNN
-	1    6550 3650
+P 6550 3450
+F 0 "#PWR0110" H 6550 3200 50  0001 C CNN
+F 1 "GND" V 6555 3322 50  0000 R CNN
+F 2 "" H 6550 3450 50  0001 C CNN
+F 3 "" H 6550 3450 50  0001 C CNN
+	1    6550 3450
 	0    1    1    0
 $EndComp
@@
 L power:GND #PWR0112
 U 1 1 6485CF38
-P 6250 3100
-F 0 "#PWR0112" H 6250 2850 50  0001 C CNN
-F 1 "GND" V 6255 2972 50  0000 R CNN
-F 2 "" H 6250 3100 50  0001 C CNN
-F 3 "" H 6250 3100 50  0001 C CNN
-	1    6250 3100
+P 6350 2550
+F 0 "#PWR0112" H 6350 2300 50  0001 C CNN
+F 1 "GND" V 6355 2422 50  0000 R CNN
+F 2 "" H 6350 2550 50  0001 C CNN
+F 3 "" H 6350 2550 50  0001 C CNN
+	1    6350 2550
 	0    1    1    0
 $EndComp
@@
 Text GLabel 5800 3350 2    50   Input ~ 0
 SERVO
-Text GLabel 6000 1950 0    50   Input ~ 0
+Text GLabel 6100 1300 0    50   Input ~ 0
 SCL
-Text GLabel 6000 2050 0    50   Input ~ 0
+Text GLabel 6100 1400 0    50   Input ~ 0
 SDA
-Text GLabel 6250 2900 0    50   Input ~ 0
+Text GLabel 6350 2350 0    50   Input ~ 0
 SERVO
 $Comp
@@
 Wire Wire Line
 	6200 4000 6550 4000
-NoConn ~ 5800 3250
+NoConn ~ 5800 3450
 NoConn ~ 5800 3150
 NoConn ~ 5800 3050
-NoConn ~ 5800 2950
 NoConn ~ 5800 2850
+NoConn ~ 5800 2750
 NoConn ~ 4600 2350
 NoConn ~ 4600 2550
@@
 NoConn ~ 4600 3750
 NoConn ~ 4600 3850
-NoConn ~ 6400 1750
+NoConn ~ 6500 1100
 $Comp
 L Device:Battery BT1
@@
 	0    -1   -1   0
 $EndComp
-Wire Wire Line
-	5800 3450 6550 3450
 NoConn ~ 4600 2850
 NoConn ~ 4600 2950
 NoConn ~ 4600 3050
+Wire Wire Line
+	6550 3250 5800 3250
+$Comp
+L LoRa32U4:LoRa32U4 U1
+U 1 1 64BFF81C
+P 5200 2750
+F 0 "U1" H 5200 3515 50  0000 C CNN
+F 1 "LoRa32U4" H 5200 3424 50  0000 C CNN
+F 2 "MODULOS:Lora32U4" H 5200 2750 50  0001 C CNN
+F 3 "" H 5200 2750 50  0001 C CNN
+	1    5200 2750
+	1    0    0    -1
+$EndComp
+$Comp
+L power:+5V #PWR0118
+U 1 1 64C03C45
+P 5800 2950
+F 0 "#PWR0118" H 5800 2800 50  0001 C CNN
+F 1 "+5V" V 5815 3078 50  0000 L CNN
+F 2 "" H 5800 2950 50  0001 C CNN
+F 3 "" H 5800 2950 50  0001 C CNN
+	1    5800 2950
+	0    1    1    0
+$EndComp
 $EndSCHEMATC

Commit message: Correccion pcb
Parts:
- removed BT1: 9V, TerminalBlock_Phoenix:TerminalBlock_Phoenix_MKDS-1,5-2-5.08_1x02_P5.08mm_Horizontal, symbol Device:Battery
- removed R1, R3: 100, Resistor_THT:R_Axial_DIN0207_L6.3mm_D2.5mm_P10.16mm_Horizontal, symbol Device:R
- removed R2: 180, Resistor_THT:R_Axial_DIN0207_L6.3mm_D2.5mm_P10.16mm_Horizontal, symbol Device:R
- removed R4: 220, Resistor_THT:R_Axial_DIN0207_L6.3mm_D2.5mm_P10.16mm_Horizontal, symbol Device:R
Changed lines of the file:
@@
 NoConn ~ 6500 1100
-$Comp
-L Device:Battery BT1
-U 1 1 64B82FDD
-P 3200 1450
-F 0 "BT1" H 3308 1496 50  0000 L CNN
-F 1 "9V" H 3250 1300 50  0000 L CNN
-F 2 "TerminalBlock_Phoenix:TerminalBlock_Phoenix_MKDS-1,5-2-5.08_1x02_P5.08mm_Horizontal" V 3200 1510 50  0001 C CNN
-F 3 "~" V 3200 1510 50  0001 C CNN
-	1    3200 1450
-	1    0    0    -1
-$EndComp
-$Comp
-L Device:R R1
-U 1 1 64B83CB1
-P 3550 1300
-F 0 "R1" H 3620 1346 50  0000 L CNN
-F 1 "100" H 3620 1255 50  0000 L CNN
-F 2 "Resistor_THT:R_Axial_DIN0207_L6.3mm_D2.5mm_P10.16mm_Horizontal" V 3480 1300 50  0001 C CNN
-F 3 "~" H 3550 1300 50  0001 C CNN
-	1    3550 1300
-	1    0    0    -1
-$EndComp
 $Comp
 L Diode:1N4001 D1
@@
 Connection ~ 3850 3650
 $Comp
-L Device:R R2
-U 1 1 64B8C058
-P 3550 1700
-F 0 "R2" H 3620 1746 50  0000 L CNN
-F 1 "180" H 3620 1655 50  0000 L CNN
-F 2 "Resistor_THT:R_Axial_DIN0207_L6.3mm_D2.5mm_P10.16mm_Horizontal" V 3480 1700 50  0001 C CNN
-F 3 "~" H 3550 1700 50  0001 C CNN
-	1    3550 1700
-	1    0    0    -1
-$EndComp
-$Comp
-L Device:R R4
-U 1 1 64B8C9C1
-P 3900 2000
-F 0 "R4" H 3970 2046 50  0000 L CNN
-F 1 "220" H 3970 1955 50  0000 L CNN
-F 2 "Resistor_THT:R_Axial_DIN0207_L6.3mm_D2.5mm_P10.16mm_Horizontal" V 3830 2000 50  0001 C CNN
-F 3 "~" H 3900 2000 50  0001 C CNN
-	1    3900 2000
-	1    0    0    -1
-$EndComp
-Wire Wire Line
-	3200 1250 3200 1150
-Wire Wire Line
-	3200 1650 3200 1850
-Wire Wire Line
-	3200 1150 3550 1150
-Wire Wire Line
-	3200 1850 3550 1850
-Wire Wire Line
-	3550 1850 3550 2150
-Wire Wire Line
-	3550 2150 3900 2150
-Connection ~ 3550 1850
-Wire Wire Line
-	3550 1500 3550 1450
-Wire Wire Line
-	3550 1550 3550 1500
-Connection ~ 3550 1500
-$Comp
-L Device:R R3
-U 1 1 64B8C357
-P 3900 1650
-F 0 "R3" H 3970 1696 50  0000 L CNN
-F 1 "100" H 3970 1605 50  0000 L CNN
-F 2 "Resistor_THT:R_Axial_DIN0207_L6.3mm_D2.5mm_P10.16mm_Horizontal" V 3830 1650 50  0001 C CNN
-F 3 "~" H 3900 1650 50  0001 C CNN
-	1    3900 1650
-	1    0    0    -1
-$EndComp
-Wire Wire Line
-	3550 1500 3900 1500
-Wire Wire Line
-	3900 1800 3900 1850
-$Comp
-L power:+5V #PWR0115
-U 1 1 64B93850
-P 3550 1500
-F 0 "#PWR0115" H 3550 1350 50  0001 C CNN
-F 1 "+5V" V 3550 1600 50  0000 L CNN
-F 2 "" H 3550 1500 50  0001 C CNN
-F 3 "" H 3550 1500 50  0001 C CNN
-	1    3550 1500
-	0    -1   -1   0
-$EndComp
-$Comp
-L power:+3.3V #PWR0116
-U 1 1 64B93E40
-P 3900 1800
-F 0 "#PWR0116" H 3900 1650 50  0001 C CNN
-F 1 "+3.3V" V 3915 1928 50  0000 L CNN
-F 2 "" H 3900 1800 50  0001 C CNN
-F 3 "" H 3900 1800 50  0001 C CNN
-	1    3900 1800
-	0    1    1    0
-$EndComp
-Connection ~ 3900 1800
-$Comp
 L power:+3.3V #PWR0117

Commit message: Cambio de fuente
Parts:
- added J1: Conn_01x02, TerminalBlock_Phoenix:TerminalBlock_Phoenix_MKDS-1,5-2_1x02_P5.00mm_Horizontal, symbol Connector_Generic:Conn_01x02
- added U3: LD1117S33TR_SOT223, Package_TO_SOT_THT:TO-220-3_Vertical, symbol Regulator_Linear:LD1117S33TR_SOT223
- added U4: LM7805_TO220, Package_TO_SOT_THT:TO-220-3_Vertical, symbol Regulator_Linear:LM7805_TO220
Connections:
- net +3V3: now also U3.3 (VI)
- net +5V: now also U3.2 (VO), U4.1 (VI)
- net GND: now also J1.2 (Pin_2), U3.1 (GND), U4.2 (GND)
- new net: J1.1 (Pin_1), U4.3 (VO)
Changed lines of the file:
@@
 	0    1    1    0
 $EndComp
+$Comp
+L Regulator_Linear:LM7805_TO220 U4
+U 1 1 651AE70B
+P 4350 1350
+F 0 "U4" H 4350 1592 50  0000 C CNN
+F 1 "LM7805_TO220" H 4350 1501 50  0000 C CNN
+F 2 "Package_TO_SOT_THT:TO-220-3_Vertical" H 4350 1575 50  0001 C CIN
+F 3 "https://www.onsemi.cn/PowerSolutions/document/MC7800-D.PDF" H 4350 1300 50  0001 C CNN
+	1    4350 1350
+	1    0    0    -1
+$EndComp
+$Comp
+L Regulator_Linear:LD1117S33TR_SOT223 U3
+U 1 1 651AF6C9
+P 3550 1350
+F 0 "U3" H 3550 1592 50  0000 C CNN
+F 1 "LD1117S33TR_SOT223" H 3550 1501 50  0000 C CNN
+F 2 "Package_TO_SOT_THT:TO-220-3_Vertical" H 3550 1550 50  0001 C CNN
+F 3 "http://www.st.com/st-web-ui/static/active/en/resource/technical/document/datasheet/CD00000544.pdf" H 3650 1100 50  0001 C CNN
+	1    3550 1350
+	1    0    0    -1
+$EndComp
+$Comp
+L Connector_Generic:Conn_01x02 J1
+U 1 1 651B1155
+P 5100 1350
+F 0 "J1" H 5180 1342 50  0000 L CNN
+F 1 "Conn_01x02" H 5180 1251 50  0000 L CNN
+F 2 "TerminalBlock_Phoenix:TerminalBlock_Phoenix_MKDS-1,5-2_1x02_P5.00mm_Horizontal" H 5100 1350 50  0001 C CNN
+F 3 "~" H 5100 1350 50  0001 C CNN
+	1    5100 1350
+	1    0    0    -1
+$EndComp
+Wire Wire Line
+	4900 1350 4650 1350
+Wire Wire Line
+	4900 1450 4800 1450
+Wire Wire Line
+	4800 1450 4800 1650
+Wire Wire Line
+	4800 1650 4350 1650
+Wire Wire Line
+	3550 1650 3950 1650
+Connection ~ 4350 1650
+Wire Wire Line
+	3850 1350 3950 1350
+$Comp
+L power:+5V #PWR0115
+U 1 1 651B70A7
+P 3950 1350
+F 0 "#PWR0115" H 3950 1200 50  0001 C CNN
+F 1 "+5V" H 3965 1523 50  0000 C CNN
+F 2 "" H 3950 1350 50  0001 C CNN
+F 3 "" H 3950 1350 50  0001 C CNN
+	1    3950 1350
+	1    0    0    -1
+$EndComp
+Connection ~ 3950 1350
+Wire Wire Line
+	3950 1350 4050 1350
+$Comp
+L power:GND #PWR0116
+U 1 1 651B75A5
+P 3950 1650
+F 0 "#PWR0116" H 3950 1400 50  0001 C CNN
+F 1 "GND" H 3955 1477 50  0000 C CNN
+F 2 "" H 3950 1650 50  0001 C CNN
+F 3 "" H 3950 1650 50  0001 C CNN
+	1    3950 1650
+	1    0    0    -1
+$EndComp
+Connection ~ 3950 1650
+Wire Wire Line
+	3950 1650 4350 1650
+$Comp
+L power:+3.3V #PWR0119
+U 1 1 651B78BF
+P 3250 1350
+F 0 "#PWR0119" H 3250 1200 50  0001 C CNN
+F 1 "+3.3V" V 3265 1478 50  0000 L CNN
+F 2 "" H 3250 1350 50  0001 C CNN
+F 3 "" H 3250 1350 50  0001 C CNN
+	1    3250 1350
+	0    -1   -1   0
+$EndComp
 $EndSCHEMATC
