File: DispenM/Balanza/Dispen2/Dispen2.sch (KiCad schematic (older format))
At the start: 11 parts, among them J1 Conn_01x02, M1 Motor_Servo, U1 LoRa32U4, U2 DS3231MZ, U3 LD1117S33TR_SOT223, U4 LM7805_TO220

Commit message: Ok sensor Hu
Connections:
- net +3V3: now also U3.2 (VO); no longer U3.3 (VI)
- net +5V: now also NiHALL1.2 (Pin_2), U3.3 (VI), U4.3 (VO); no longer NiHALL1.3 (Pin_3), U3.2 (VO), U4.1 (VI)
- net GND: now also NiHALL1.3 (Pin_3); no longer NiHALL1.2 (Pin_2)
- net at J1.1 (Pin_1): now also U4.1 (VI); no longer U4.3 (VO)
Other:
- moved on the sheet: U3, U4
Changed lines of the file:
@@
 L power:GND #PWR0107
 U 1 1 6485A77A
-P 4050 2850
-F 0 "#PWR0107" H 4050 2600 50  0001 C CNN
-F 1 "GND" V 4055 2722 50  0000 R CNN
-F 2 "" H 4050 2850 50  0001 C CNN
-F 3 "" H 4050 2850 50  0001 C CNN
-	1    4050 2850
+P 4050 2950
+F 0 "#PWR0107" H 4050 2700 50  0001 C CNN
+F 1 "GND" V 4055 2822 50  0000 R CNN
+F 2 "" H 4050 2950 50  0001 C CNN
+F 3 "" H 4050 2950 50  0001 C CNN
+	1    4050 2950
 	0    -1   -1   0
 $EndComp
@@
 L power:+5V #PWR0113
 U 1 1 6485D4A5
-P 4050 2950
-F 0 "#PWR0113" H 4050 2800 50  0001 C CNN
-F 1 "+5V" V 4065 3078 50  0000 L CNN
-F 2 "" H 4050 2950 50  0001 C CNN
-F 3 "" H 4050 2950 50  0001 C CNN
-	1    4050 2950
+P 4050 2850
+F 0 "#PWR0113" H 4050 2700 50  0001 C CNN
+F 1 "+5V" V 4065 2978 50  0000 L CNN
+F 2 "" H 4050 2850 50  0001 C CNN
+F 3 "" H 4050 2850 50  0001 C CNN
+	1    4050 2850
 	0    1    1    0
 $EndComp
@@
 L Regulator_Linear:LM7805_TO220 U4
 U 1 1 651AE70B
-P 4350 1350
-F 0 "U4" H 4350 1592 50  0000 C CNN
-F 1 "LM7805_TO220" H 4350 1501 50  0000 C CNN
-F 2 "Package_TO_SOT_THT:TO-220-3_Vertical" H 4350 1575 50  0001 C CIN
-F 3 "https://www.onsemi.cn/PowerSolutions/document/MC7800-D.PDF" H 4350 1300 50  0001 C CNN
-	1    4350 1350
-	1    0    0    -1
+P 4450 1350
+F 0 "U4" H 4450 1592 50  0000 C CNN
+F 1 "LM7805_TO220" H 4450 1501 50  0000 C CNN
+F 2 "Package_TO_SOT_THT:TO-220-3_Vertical" H 4450 1575 50  0001 C CIN
+F 3 "https://www.onsemi.cn/PowerSolutions/document/MC7800-D.PDF" H 4450 1300 50  0001 C CNN
+	1    4450 1350
+	-1   0    0    -1
 $EndComp
 $Comp
 L Regulator_Linear:LD1117S33TR_SOT223 U3
 U 1 1 651AF6C9
-P 3550 1350
-F 0 "U3" H 3550 1592 50  0000 C CNN
-F 1 "LD1117S33TR_SOT223" H 3550 1501 50  0000 C CNN
-F 2 "Package_TO_SOT_THT:TO-220-3_Vertical" H 3550 1550 50  0001 C CNN
-F 3 "http://www.st.com/st-web-ui/static/active/en/resource/technical/document/datasheet/CD00000544.pdf" H 3650 1100 50  0001 C CNN
-	1    3550 1350
-	1    0    0    -1
+P 3050 1350
+F 0 "U3" H 3050 1592 50  0000 C CNN
+F 1 "LD1117S33TR_SOT223" H 3050 1501 50  0000 C CNN
+F 2 "Package_TO_SOT_THT:TO-220-3_Vertical" H 3050 1550 50  0001 C CNN
+F 3 "http://www.st.com/st-web-ui/static/active/en/resource/technical/document/datasheet/CD00000544.pdf" H 3150 1100 50  0001 C CNN
+	1    3050 1350
+	-1   0    0    -1
 $EndComp
 $Comp
@@
 	1    0    0    -1
 $EndComp
-Wire Wire Line
-	4900 1350 4650 1350
-Wire Wire Line
-	4900 1450 4800 1450
-Wire Wire Line
-	4800 1450 4800 1650
-Wire Wire Line
-	4800 1650 4350 1650
-Wire Wire Line
-	3550 1650 3950 1650
-Connection ~ 4350 1650
-Wire Wire Line
-	3850 1350 3950 1350
-$Comp
-L power:+5V #PWR0115
-U 1 1 651B70A7
-P 3950 1350
-F 0 "#PWR0115" H 3950 1200 50  0001 C CNN
-F 1 "+5V" H 3965 1523 50  0000 C CNN
-F 2 "" H 3950 1350 50  0001 C CNN
-F 3 "" H 3950 1350 50  0001 C CNN
-	1    3950 1350
-	1    0    0    -1
-$EndComp
-Connection ~ 3950 1350
-Wire Wire Line
-	3950 1350 4050 1350
 $Comp
 L power:GND #PWR0116
@@
 $EndComp
 Connection ~ 3950 1650
-Wire Wire Line
-	3950 1650 4350 1650
 $Comp
 L power:+3.3V #PWR0119
 U 1 1 651B78BF
-P 3250 1350
-F 0 "#PWR0119" H 3250 1200 50  0001 C CNN
-F 1 "+3.3V" V 3265 1478 50  0000 L CNN
-F 2 "" H 3250 1350 50  0001 C CNN
-F 3 "" H 3250 1350 50  0001 C CNN
-	1    3250 1350
-	0    -1   -1   0
-$EndComp
+P 2750 1350
+F 0 "#PWR0119" H 2750 1200 50  0001 C CNN
+F 1 "+3.3V" V 2765 1478 50  0000 L CNN
+F 2 "" H 2750 1350 50  0001 C CNN
+F 3 "" H 2750 1350 50  0001 C CNN
+	1    2750 1350
+	0    -1   -1   0
+$EndComp
+Wire Wire Line
+	3950 1650 4450 1650
+Wire Wire Line
+	3050 1650 3950 1650
+Wire Wire Line
+	4450 1650 4900 1650
+Wire Wire Line
+	4900 1650 4900 1450
+Connection ~ 4450 1650
+Wire Wire Line
+	4750 1350 4900 1350
+Wire Wire Line
+	4150 1350 3750 1350
+$Comp
+L power:+5V #PWR0115
+U 1 1 65257AC4
+P 3750 1350
+F 0 "#PWR0115" H 3750 1200 50  0001 C CNN
+F 1 "+5V" H 3765 1523 50  0000 C CNN
+F 2 "" H 3750 1350 50  0001 C CNN
+F 3 "" H 3750 1350 50  0001 C CNN
+	1    3750 1350
+	1    0    0    -1
+$EndComp
+Connection ~ 3750 1350
+Wire Wire Line
+	3750 1350 3350 1350
 $EndSCHEMATC

Commit message: nuevo circuito
nuevo circuito
Parts:
- added CABLE1, CABLE2: R, Resistor_THT:R_Axial_DIN0411_L9.9mm_D3.6mm_P20.32mm_Horizontal, symbol Device:R
Connections:
- net GND: now also CABLE1.1, CABLE1.2, CABLE2.1, CABLE2.2
Changed lines of the file:
@@
 Wire Wire Line
 	3750 1350 3350 1350
+$Comp
+L Device:R CABLE1
+U 1 1 654A6BE8
+P 5000 4300
+F 0 "CABLE1" V 4793 4300 50  0000 C CNN
+F 1 "R" V 4884 4300 50  0000 C CNN
+F 2 "Resistor_THT:R_Axial_DIN0411_L9.9mm_D3.6mm_P20.32mm_Horizontal" V 4930 4300 50  0001 C CNN
+F 3 "~" H 5000 4300 50  0001 C CNN
+	1    5000 4300
+	0    1    1    0
+$EndComp
+$Comp
+L power:GND #PWR0120
+U 1 1 654A7900
+P 4850 4300
+F 0 "#PWR0120" H 4850 4050 50  0001 C CNN
+F 1 "GND" V 4855 4172 50  0000 R CNN
+F 2 "" H 4850 4300 50  0001 C CNN
+F 3 "" H 4850 4300 50  0001 C CNN
+	1    4850 4300
+	0    1    1    0
+$EndComp
+$Comp
+L power:GND #PWR0121
+U 1 1 654A812A
+P 5150 4300
+F 0 "#PWR0121" H 5150 4050 50  0001 C CNN
+F 1 "GND" H 5155 4127 50  0000 C CNN
+F 2 "" H 5150 4300 50  0001 C CNN
+F 3 "" H 5150 4300 50  0001 C CNN
+	1    5150 4300
+	0    -1   -1   0
+$EndComp
+$Comp
+L Device:R CABLE2
+U 1 1 654B1BB8
+P 5000 4650
+F 0 "CABLE2" V 4793 4650 50  0000 C CNN
+F 1 "R" V 4884 4650 50  0000 C CNN
+F 2 "Resistor_THT:R_Axial_DIN0411_L9.9mm_D3.6mm_P20.32mm_Horizontal" V 4930 4650 50  0001 C CNN
+F 3 "~" H 5000 4650 50  0001 C CNN
+	1    5000 4650
+	0    1    1    0
+$EndComp
+$Comp
+L power:GND #PWR0122
+U 1 1 654B214E
+P 4850 4650
+F 0 "#PWR0122" H 4850 4400 50  0001 C CNN
+F 1 "GND" V 4855 4522 50  0000 R CNN
+F 2 "" H 4850 4650 50  0001 C CNN
+F 3 "" H 4850 4650 50  0001 C CNN
+	1    4850 4650
+	0    1    1    0
+$EndComp
+$Comp
+L power:GND #PWR0123
+U 1 1 654B2579
+P 5150 4650
+F 0 "#PWR0123" H 5150 4400 50  0001 C CNN
+F 1 "GND" H 5155 4477 50  0000 C CNN
+F 2 "" H 5150 4650 50  0001 C CNN
+F 3 "" H 5150 4650 50  0001 C CNN
+	1    5150 4650
+	0    -1   -1   0
+$EndComp
 $EndSCHEMATC
