File: DispenM/DispenM2/DispenGSM.sch (EAGLE design)
At the start: 16 parts, among them IC1 7805TV, IC3 LM1117T-3.3-V, X1 SMKDSP_1,5/2, X2 SMKDSP_1,5/2, X3 SMKDSP_1,5/2

Commit message: 27/11/2024
Actualizacion circuito
Parts:
- removed C1: 10U, rcl:CPOL-EUTT2D6
- removed C2: 0.33U, rcl:CPOL-EUTT2D6
- removed C3: 0.1U, rcl:CPOL-EUTT2D6
- removed U$2: SIM800L, SIM800L:SIM800L
- removed X2, X3: SMKDSP_1,5/2, con-phoenix-smkdsp:SMKDSP_1,5/2
- added D1: 1N4004, diode:1N4004
- added JP1: (no value), pinhead:PINHD-1X6
Connections:
- removed net +12V: C2.+, IC1.VI, X1-1.KL
- new net N$1: IC1.VI, X1-1.KL
- new net N$2: D1.C, JP1.2
- new net RXD2: JP1.4, U$1.GPIO17
- new net TXD2: JP1.5, U$1.GPIO16
- net +3V3: now also SHARP.2; no longer C1.+, SHARP.3, X2-1.KL
- net +5V: now also D1.A; no longer C3.+, U$1.5V, U$2.VCC, X3-1.KL
- net DATOB1: now also U$1.GPIO34(ADC1_6)
- net DATOB2: now also U$1.GPIO35(ADC1_7)
- net GND: now also JP1.6, SHARP.3; no longer C1.-, C2.-, C3.-, SHARP.2, U$2.GND, X2-2.KL, X3-2.KL
- net RXD: no longer U$2.RXD
- net SCK2: now also U$1.GPIO14(ADC2_6/MTMSHSPI_SCK)
- net SDA2: now also U$1.GPIO4(ADC2_0)
- net SERVO: now also U$1.GPIO32(ADC1_4)
- net SHARP: now also U$1.GPIO27(ADC2_7)
- net TXD: no longer U$2.TXD
Other:
- moved on the sheet: IC1, X1-1, X1-2
